File: hardware/bonsai_pcb/bonsai_pcb.kicad_pcb (KiCad board)
At the start: 2 copper layers, 53 x 23 mm, 6 parts, among them J1 Audio Amp Conn, J2 BAT +, J3 Battery Pin Socket, J4 BAT -, SW1 BT1, U1 XIAO-ESP32-S3-SMD

Commit message: Update PCB and BOM files
Parts:
- removed J2: BAT +, Connector_Wire:SolderWirePad_1x01_SMD_2x4mm
- removed J4: BAT -, Connector_Wire:SolderWirePad_1x01_SMD_2x4mm
- added B+: B+ Wire, Connector_Wire:SolderWirePad_1x01_SMD_2x4mm, B.Cu at (159.9, 105.7)
- added G***: LOGO, assets:bonsai-icon, B.Cu at (135.0, 94.1)
- J3: value Battery Pin Socket -> PH2.0 Battery Connector
- moved J3 0.10 mm to (168.9, 99.4)
Connections:
- J3 pad 1: Net-(J3-Pin_1) -> GND
Routing:
- net GND: track 39.9 -> 2.58 mm, vias 16 -> 17
- net Net-(J3-Pin_1): track 5.13 -> 0.00 mm
- net Net-(J2-Pin_1): track 13.9 -> 16.9 mm
- net VIN: track 33.7 -> 33.0 mm
- added copper zone on B.Cu, net GND
Other:
- outline, holes or cut-outs redrawn
- board text added: "->"
- board text added: "SOLDER HERE"
- board text added: "v0.1 23/07/26 Biel Vazquez Mata"
- board text added: "⌈ ⌉ MAX98357 ⌊ ⌋"
