File: hardware/bonsai_pcb/bonsai_pcb.kicad_sch (KiCad schematic)
At the start: 6 parts, among them J1 Audio Amp Conn, J2 BAT +, J3 Battery Pin Socket, J4 BAT -, SW1 BT1, U1 XIAO-ESP32-S3-SMD

Commit message: Update PCB and BOM files
Parts:
- removed J3: Battery Pin Socket, Connector_JST:JST_PH_S2B-PH-K_1x02_P2.00mm_Horizontal, symbol Connector:Conn_01x02_Pin
- removed J4: BAT -, symbol Connector:Conn_01x01_Socket
- added J3: PH2.0 Battery Connector, Connector_JST:JST_PH_S2B-PH-K_1x02_P2.00mm_Horizontal, symbol Connector:Conn_01x02_Socket
- J2: value BAT + -> B+ Wire; footprint (none) -> Connector_Wire:SolderWirePad_1x01_SMD_2x4mm
Connections:
- net GND: now also U1.33 (GND), J3.1 (Pin_1)
- net at J2.1 (Pin_1): now also J3.2 (Pin_2)
